File: BQ40Z80.kicad_pcb (KiCad board)
At the start: 4 copper layers, 69 x 46 mm, 95 parts, among them J1 Conn_01x02, J2 Conn_01x03, J3 Conn_01x06_MountingPin, J4 Conn_01x08, J5 Conn_01x02_MountingPin, Q1 AO3401A, Q10 AON6411, Q11 2N7002, Q12 CSD18540Q5B, Q2 AO3401A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

Commit message: 1
Routing:
- net Net-(Q8-G): vias 3 -> 2
- net Net-(Q12-D): vias 2 -> 34
- net Net-(C9-Pad1): vias 26 -> 96
- net Net-(C11-Pad1): vias 1 -> 0
- net GND: vias 75 -> 121
- net /BAT+: vias 69 -> 98
- net (no net): vias 350 -> 0
- added copper zone on B.Cu, net /PACK+
- added copper zone on In1.Cu, net /PACK+
- added copper zone on In2.Cu, net /PACK+
- added copper zone on B.Cu, net /PACK-
- added copper zone on In1.Cu, net /PACK-
- added copper zone on In2.Cu, net /PACK-
- added copper zone on B.Cu, net Net-(Q12-D)
- added copper zone on In1.Cu, net Net-(Q12-D)
- added copper zone on In2.Cu, net Net-(Q12-D)

Commit message: 1
Parts:
- removed TP8: BAT-, BQ40Z80_Footprints:SolderWirePad_1x01_SMD_14x6mm
- added NT1: NetTie_2, NetTie:NetTie-2_SMD_Pad0.5mm, F.Cu at (158.1, 122.9)
- added NT2: NetTie_2, NetTie:NetTie-2_SMD_Pad0.5mm, F.Cu at (177.0, 140.5)
- J3: value Conn_01x06_MountingPin -> Conn_01x07_MountingPin; footprint Connector_JST:JST_PH_S6B-PH-SM4-TB_1x06-1MP_P2.00mm_Horizontal -> Connector_JST:JST_PH_S7B-PH-SM4-TB_1x07-1MP_P2.00mm_Horizontal
- moved R15 7.05 mm to (137.9, 108.4), turned to 0 degrees
- moved R14 5.15 mm to (133.9, 110.2), turned to -90 degrees
- moved C7 4.40 mm to (135.4, 110.2), turned to -90 degrees
- moved Q7 1.76 mm to (131.1, 110.2), turned to 0 degrees
- moved J3 0.99 mm to (148.1, 141.0)
Connections:
- C6 pad 2: GND -> /0.0V
- R22 pad 2: GND -> GNDPWR
- R24 pad 1: GND -> GNDPWR
- R6 pad 2: GND -> /0.0V
Routing:
- net /PIN15: track 12.7 -> 36.8 mm, vias 1 -> 2
- net /0.0V: track 0.00 -> 17.9 mm
- net /PIN17: track 10.4 -> 20.8 mm, vias 1 -> 3
- net /FUSE: track 0.00 -> 8.00 mm
- net /DISP: track 0.00 -> 4.09 mm
- net GNDPWR: track 0.00 -> 3.39 mm, vias 0 -> 5
- net GND: track 3.39 -> 0.00 mm, vias 121 -> 162
- net Net-(Q7-G): track 7.75 -> 9.06 mm
- net Net-(Q7-D): track 35.1 -> 35.9 mm
- net /PIN16: track 37.0 -> 37.6 mm
- net /PACK+: track 22.0 -> 22.1 mm, vias 2 -> 18
- net /PACK-: vias 0 -> 16

Commit message: Add readme.md
Parts:
- added TP11: BAT-, BQ40Z80_Footprints:SolderWirePad_1x01_SMD_14x6mm, F.Cu at (103.5, 134.5)
- NT2: footprint NetTie:NetTie-2_SMD_Pad0.5mm -> BQ40Z80_Footprints:NetTie-2-234Layers_SMD_Pad0.5mm
- moved NT2 70.3 mm to (108.5, 124.8), turned to -90 degrees
Routing:
- net GNDPWR: vias 5 -> 112
- net GND: vias 162 -> 59
- added copper zone on B.Cu, net GNDPWR
- added copper zone on F.Cu, net GNDPWR
- added copper zone on In1.Cu, net GNDPWR
- added copper zone on In2.Cu, net GNDPWR
