File: BQ40Z80.kicad_sch (KiCad schematic)
At the start: 103 parts, among them J1 Conn_01x02, J2 Conn_01x03, J3 Conn_01x06_MountingPin, J4 Conn_01x08, J5 Conn_01x02_MountingPin, Q1 AO3401A, Q10 AON6411, Q11 2N7002, Q12 CSD18540Q5B, Q2 AO3401A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

Commit message: 1
Parts:
- removed J3: Conn_01x06_MountingPin, Connector_JST:JST_PH_S6B-PH-SM4-TB_1x06-1MP_P2.00mm_Horizontal, symbol Connector_Generic_MountingPin:Conn_01x06_MountingPin
- removed TP4: BAT-, BQ40Z80_Footprints:SolderWirePad_1x01_SMD_14x6mm, symbol Connector:TestPoint
- added J3: Conn_01x07_MountingPin, Connector_JST:JST_PH_S7B-PH-SM4-TB_1x07-1MP_P2.00mm_Horizontal, symbol Connector_Generic_MountingPin:Conn_01x07_MountingPin
- added NT1, NT2: NetTie_2, NetTie:NetTie-2_SMD_Pad0.5mm, symbol Device:NetTie_2
- added TP5: 0.0V, BQ40Z80_Footprints:TestPoint_Pad_1.0x2.0mm, symbol Connector:TestPoint
Connections:
- net 12.6V: now also J3.4 (Pin_4)
- net 16.8V: now also J3.3 (Pin_3)
- net 21.0V: now also J3.2 (Pin_2)
- net 25.2V: now also J3.1 (Pin_1)
- net 4.2V: now also J3.6 (Pin_6)
- net 8.4V: now also J3.5 (Pin_5)
- net GND: now also J3.MP (MountPin), NT1.2, NT2.1; no longer C11.2, R6.2, R6.2, R8.1
- new net 0.0V: C11.2, J3.7 (Pin_7), NT1.1, R6.2, TP5.1
- new net GNDPWR: NT2.2, R6.2, R8.1

Commit message: Add readme.md
Parts:
- added TP8: BAT-, BQ40Z80_Footprints:SolderWirePad_1x01_SMD_14x6mm, symbol Connector:TestPoint
- J5: symbol Connector_Generic_MountingPin:Conn_01x02_MountingPin -> Connector_Generic:Conn_01x02
- NT2: footprint NetTie:NetTie-2_SMD_Pad0.5mm -> BQ40Z80_Footprints:NetTie-2-234Layers_SMD_Pad0.5mm
Connections:
- net GNDPWR: now also TP8.1
Changed lines of the file:
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@@
   (junction (at 49.53 233.68) (diameter 0) (color 0 0 0 0)
   )
+  (junction (at 106.68 242.57) (diameter 0) (color 0 0 0 0)
+  )
   (junction (at 67.31 104.14) (diameter 0) (color 0 0 0 0)
   )
@@
       (effects (font (size 1.27 1.27)))
     )
-    (property "Footprint" "NetTie:NetTie-2_SMD_Pad0.5mm" (at 104.14 242.57 0)
+    (property "Footprint" "BQ40Z80_Footprints:NetTie-2-234Layers_SMD_Pad0.5mm" (at 104.14 242.57 0)
       (effects (font (size 1.27 1.27)) hide)
     )
@@
     )
   )
+  (symbol (lib_id "Connector:TestPoint") (at 106.68 242.57 0) (unit 1)
+    (in_bom yes) (on_board yes) (dnp no)
+    (property "Reference" "TP8" (at 111.76 239.268 90)
+      (effects (font (size 1.27 1.27)) hide)
+    )
+    (property "Value" "BAT-" (at 104.14 237.49 0)
+      (effects (font (size 1.27 1.27)) (justify left))
+    )
+    (property "Footprint" "BQ40Z80_Footprints:SolderWirePad_1x01_SMD_14x6mm" (at 111.76 242.57 0)
+      (effects (font (size 1.27 1.27)) hide)
+    )
+    (property "Datasheet" "~" (at 111.76 242.57 0)
+      (effects (font (size 1.27 1.27)) hide)
+    )
+    (pin "1")
+    (instances
+      (project "IP5389-BQ77915-POWER-BANK"
+        (path "/4a1f87ac-9b28-460b-85cc-06755639df63"
+          (reference "TP8") (unit 1)
+        )
+      )
+      (project "BQ40Z80"
+        (path "/61db2e73-87f8-4cdc-8474-b79ca2905d06"
+          (reference "TP11") (unit 1)
+        )
+      )
+    )
+  )
   (symbol (lib_id "Connector_Generic_MountingPin:Conn_01x07_MountingPin") (at 52.07 259.08 0) (unit 1)
     (in_bom yes) (on_board yes) (dnp no) (fields_autoplaced)
@@
     )
   )
-  (symbol (lib_id "Connector_Generic_MountingPin:Conn_01x02_MountingPin") (at 256.54 264.16 0) (unit 1)
+  (symbol (lib_id "Connector_Generic:Conn_01x02") (at 256.54 264.16 0) (unit 1)
     (in_bom yes) (on_board yes) (dnp no) (fields_autoplaced)
     (property "Reference" "J5" (at 259.08 264.5156 0)
@@
     (pin "1")
     (pin "2")
-    (pin "MP")
     (instances
       (project "BQ40Z80"
